File: board-files/rc-driver.brd (EAGLE design)
At the start: 25 x 14 mm, 15 parts, among them IC1 TINY22S

Commit message: Moving single board files to different folder.
Parts:
- R3: value (none) -> 5600
- R5: value (none) -> 1300
Changed lines of the file:
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@@
 <?xml version="1.0" encoding="utf-8"?>
 <!DOCTYPE eagle SYSTEM "eagle.dtd">
-<eagle version="7.1.0">
+<eagle version="7.2.0">
 <drawing>
 <settings>
@@
 <element name="U$1" library="mgregg" package="SO-8EP" value="A4950-HBRIDGE" x="11.5" y="6.9" rot="MR90"/>
 <element name="R2" library="resistor" package="R0805W" value="" x="17" y="6.1" rot="MR0"/>
-<element name="R3" library="resistor" package="R0603" value="" x="6.3" y="4.5" rot="MR0"/>
-<element name="R5" library="resistor" package="R0603" value="" x="6.3" y="2.9" rot="MR180"/>
+<element name="R3" library="resistor" package="R0603" value="5600" x="6.3" y="4.5" rot="MR0"/>
+<element name="R5" library="resistor" package="R0603" value="1300" x="6.3" y="2.9" rot="MR180"/>
 <element name="R6" library="resistor" package="R0603" value="" x="3.8" y="1.1" rot="MR0"/>
 </elements>
