File: board-files/rc-driver-dual.brd (EAGLE design)
At the start: 29.6 x 17.5 mm, 20 parts

Commit message: Moving single board files to different folder.
Parts:
- R3: value (none) -> 5600
- R4: value (none) -> 1300
Changed lines of the file:
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@@
 <element name="R1" library="resistor" package="R0805W" value="" x="21.068" y="6.68" rot="MR180"/>
 <element name="R2" library="resistor" package="R0805W" value="" x="21.092" y="9.508" rot="MR180"/>
-<element name="R3" library="resistor" package="R0603" value="" x="12.819" y="14.589" rot="MR0"/>
-<element name="R4" library="resistor" package="R0603" value="" x="9.6" y="13.7" rot="MR0"/>
+<element name="R3" library="resistor" package="R0603" value="5600" x="12.819" y="14.589" rot="MR0"/>
+<element name="R4" library="resistor" package="R0603" value="1300" x="9.6" y="13.7" rot="MR0"/>
 <element name="R5" library="resistor" package="R0603" value="" x="15.875" y="1.524"/>
 <element name="LED1" library="led" package="CHIPLED_0603" value="" x="20.066" y="1.27" rot="R270"/>

Commit message: Changes for battlebot competition.   More part information.   Changed steering and forward direction mixing.   Have one led for signal, and the other for no signal.
Parts:
- LED1: value (none) -> GREEN
- LED2: value (none) -> RED
- R1, R2: value (none) -> 0.047
- R5, R6: value (none) -> 360
Changed lines of the file:
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@@
 <element name="C2" library="resistor" package="C0603" value="0.1uf" x="18.227" y="15.478" rot="MR180"/>
 <element name="C3" library="resistor" package="C0603" value="0.1uf" x="15.725" y="3.358" rot="MR0"/>
-<element name="R1" library="resistor" package="R0805W" value="" x="21.068" y="6.68" rot="MR180"/>
-<element name="R2" library="resistor" package="R0805W" value="" x="21.092" y="9.508" rot="MR180"/>
+<element name="R1" library="resistor" package="R0805W" value="0.047" x="21.068" y="6.68" rot="MR180"/>
+<element name="R2" library="resistor" package="R0805W" value="0.047" x="21.092" y="9.508" rot="MR180"/>
 <element name="R3" library="resistor" package="R0603" value="5600" x="12.819" y="14.589" rot="MR0"/>
 <element name="R4" library="resistor" package="R0603" value="1300" x="9.6" y="13.7" rot="MR0"/>
-<element name="R5" library="resistor" package="R0603" value="" x="15.875" y="1.524"/>
-<element name="LED1" library="led" package="CHIPLED_0603" value="" x="20.066" y="1.27" rot="R270"/>
+<element name="R5" library="resistor" package="R0603" value="360" x="15.875" y="1.524"/>
+<element name="LED1" library="led" package="CHIPLED_0603" value="GREEN" x="20.066" y="1.27" rot="R270"/>
 <element name="RT1" library="resistor" package="R0603" value="" x="14.035" y="14.003" rot="R270"/>
 <element name="R7" library="resistor" package="R0603" value="" x="11.419" y="14.424" rot="R180"/>
-<element name="R6" library="resistor" package="R0603" value="" x="16.256" y="4.064" rot="R270"/>
-<element name="LED2" library="led" package="CHIPLED_0603" value="" x="20.066" y="2.667" rot="R270"/>
+<element name="R6" library="resistor" package="R0603" value="360" x="16.256" y="4.064" rot="R270"/>
+<element name="LED2" library="led" package="CHIPLED_0603" value="RED" x="20.066" y="2.667" rot="R270"/>
 <element name="C4" library="resistor" package="C1206" value="10uf" x="19.812" y="9.017"/>
 <element name="C5" library="resistor" package="C0603" value="0.1uf" x="15.875" y="12.954" rot="MR0"/>
